File: Ka-band-Mixer/Ka-band-Mixer.kicad_pcb (KiCad board)
At the start: 4 copper layers, 55.9 x 41.9 mm, 75 parts, among them J1 Conn_01x02_Male, J2 Conn_01x02_Male, J3 Connector_Conn_01x02_Male, J4 Conn_01x05_Male, J5 SMA_END-frequencySintesizer, U1 ADF4150HV, U2 LT1962-3.3, U3 LT3010, U4 HMC739LP4E, U5 LT1962-5, U6 LT1962-5, U7 HMC292, X1 IQXT-220-1

Commit message: update
Routing:
- net 0: vias 97 -> 218
Other:
- board text added: "3.3V"
- board text added: "5V A"
- board text added: "5V D"
- board text added: "9V"
- board text added: "CLK"

Commit message: update
Parts:
- U7: value HMC292 -> E_12_4
