File: Ka-band-Mixer/Ka-band-Mixer.kicad_pcb (KiCad board)
At the start: 4 copper layers, 58.9 x 41.9 mm, 75 parts, among them J1 Conn_01x05_Male, J2 Conn_01x02_Male, J3 Conn_01x02_Male, J4 Connector_Conn_01x02_Male, J5 SMA_END-frequencySintesizer, U1 ADF4150HV, U2 LT3010, U3 LT1962-3.3, U4 LT1962-5, U5 LT1962-5, U6 HMC739LP4E, U7 HMC292ALC3B, X1 IQXT-220-1

Commit message: Update for DRC
Parts:
- D2, D3: footprint Diode_SMD:D_MELF -> Microwave_LO_Generator:D_MELF
- J1: footprint Connector_PinHeader_2.54mm:PinHeader_1x05_P2.54mm_Vertical -> Microwave_LO_Generator:PinHeader_1x05_P2.54mm_Vertical
- J2, J3: footprint Connector_PinHeader_2.54mm:PinHeader_1x02_P2.54mm_Vertical -> Microwave_LO_Generator:PinHeader_1x02_P2.54mm_Vertical
- TP1, TP2, TP3, TP4, TP5, TP6: footprint TestPoint:TestPoint_Loop_D2.60mm_Drill1.6mm_Beaded -> Microwave_LO_Generator:TestPoint_Loop_D2.60mm_Drill1.6mm_Beaded
- U2: footprint Package_SO:MSOP-8-1EP_3x3mm_P0.65mm_EP1.68x1.88mm -> Microwave_LO_Generator:MSOP-8-1EP_3x3mm_P0.65mm_EP1.68x1.88mm
- U3, U4, U5: footprint Package_SO:MSOP-8_3x3mm_P0.65mm -> Microwave_LO_Generator:MSOP-8_3x3mm_P0.65mm
- X1: footprint Oscillator:Oscillator_SMD_Abracon_ASE-4Pin_3.2x2.5mm_HandSoldering -> Microwave_LO_Generator:Oscillator_SMD_Abracon_ASE-4Pin_3.2x2.5mm_HandSoldering
Other:
- board size 58.9 x 41.9 mm -> 58.8 x 41.9 mm
- rule pad_to_mask_clearance: 0.2 -> 0.215
- rule solder_mask_min_width: 0.2 -> 0.215
