File: Ka-band-Mixer/frequencySynthesizer.sch (KiCad schematic (older format))
At the start: 28 parts, among them J4 Conn_01x05_Male, U1 ADF4150HV, X1 IQXT-220-1

Commit message: update bom
Parts:
- U1: Supplier Stock Code Mouser 584-ADF4150HVBCPZ -> 584-ADF4150HVBCPZ
- X1: Manufacturer/Part Number HMC292ALC3B -> IQXT-220-1; Supplier Stock Code 584-HMC292ALC3B -> LFTCXO075792Cutt
- renumbered C12 to C10, C13 to C11, C14 to C12, C15 to C13, C4 to C3, C6 to C4, C7 to C5, C8 to C6, C9 to C7, C10 to C8, C11 to C9, J4 to J1, R10 to R1, R6 to R10, R1 to R2, R18 to R3, R19 to R4, R20 to R5, R2 to R6, R3 to R7, R4 to R8, R5 to R9

Commit message: Update for DRC
Parts:
- J1: footprint Connector_PinHeader_2.54mm:PinHeader_1x05_P2.54mm_Vertical -> Microwave_LO_Generator:PinHeader_1x05_P2.54mm_Vertical
- TP1: footprint TestPoint:TestPoint_Loop_D2.60mm_Drill1.6mm_Beaded -> Microwave_LO_Generator:TestPoint_Loop_D2.60mm_Drill1.6mm_Beaded
- X1: footprint Oscillator:Oscillator_SMD_Abracon_ASE-4Pin_3.2x2.5mm_HandSoldering -> Microwave_LO_Generator:Oscillator_SMD_Abracon_ASE-4Pin_3.2x2.5mm_HandSoldering
Changed lines of the file:
@@
 F 0 "X1" H 2544 3596 50  0000 L CNN
 F 1 "IQXT-220-1" H 2544 3505 50  0000 L CNN
-F 2 "Oscillator:Oscillator_SMD_Abracon_ASE-4Pin_3.2x2.5mm_HandSoldering" H 2200 3550 50  0001 C CNN
+F 2 "Microwave_LO_Generator:Oscillator_SMD_Abracon_ASE-4Pin_3.2x2.5mm_HandSoldering" H 2200 3550 50  0001 C CNN
 F 3 "https://www.mouser.it/datasheet/2/741/LFTCXO075792Cutt-1115708.pdf" H 2200 3550 50  0001 C CNN
 F 4 "IQXT-220-1" H 2200 3550 50  0001 C CNN "Manufacturer/Part Number"
@@
 F 0 "TP1" H 3092 3476 50  0000 R CNN
 F 1 "TestPoint" H 3092 3567 50  0000 R CNN
-F 2 "TestPoint:TestPoint_Loop_D2.60mm_Drill1.6mm_Beaded" H 3350 3450 50  0001 C CNN
+F 2 "Microwave_LO_Generator:TestPoint_Loop_D2.60mm_Drill1.6mm_Beaded" H 3350 3450 50  0001 C CNN
 F 3 "https://www.mouser.it/datasheet/2/215/005-5009-741293.pdf" H 3350 3450 50  0001 C CNN
 F 4 "5007" H 3150 3450 50  0001 C CNN "Manufacturer/Part Number"
@@
 F 0 "J1" H 2858 2181 50  0000 C CNN
 F 1 "Conn_01x05_Male" H 2858 2090 50  0000 C CNN
-F 2 "Connector_PinHeader_2.54mm:PinHeader_1x05_P2.54mm_Vertical" H 2750 1800 50  0001 C CNN
+F 2 "Microwave_LO_Generator:PinHeader_1x05_P2.54mm_Vertical" H 2750 1800 50  0001 C CNN
 F 3 "~" H 2750 1800 50  0001 C CNN
 	1    2750 1800
