File: Ka-band-Mixer/powerSupply.sch (KiCad schematic (older format))
At the start: 34 parts, among them J1 Conn_01x02_Male, J2 Conn_01x02_Male, U2 LT1962-3.3, U3 LT3010, U5 LT1962-5, U6 LT1962-5

Commit message: Update BOM
Parts:
- C16: Manufacturer/Part Number GCM1555C1H101JA16D -> 963-GMK105CC6105MV-F; Supplier Stock Code Mouser 81-GCM1555C1H101JA6D -> GMK105CC6105MV-F
- C17, C19, C23: Manufacturer/Part Number GCM1555C1H101JA16D -> 0402YD475MAT2A; Supplier Stock Code Mouser 81-GCM1555C1H101JA6D -> 581-0402YD475MAT2A
- C21, C24, C31: Supplier Stock Code Mouser 81-GCM1555C1H101JA6D -> 81-GCM1555C1H101JA6D
- C22: Manufacturer/Part Number GCM1555C1H101JA16D -> GMK105CC6105MV-F; Supplier Stock Code Mouser 81-GCM1555C1H101JA6D -> 963-GMK105CC6105MV-F
- C25, C35, C36: Manufacturer/Part Number GCM1555C1H101JA16D -> C1005X5R1A335K050BC; Supplier Stock Code Mouser 81-GCM1555C1H101JA6D -> 810-C1005X5R1A335K0C
- C3, C5: Manufacturer/Part Number GCM1555C1H101JA16D -> 04025C101KAT2A; Supplier Stock Code Mouser 81-GCM1555C1H101JA6D -> 581-04025C101KAT2A
- C32, C33, C34: Manufacturer/Part Number GCM1555C1H101JA16D -> 0402YC103KAT4A; Supplier Stock Code Mouser 81-GCM1555C1H101JA6D -> 581-0402YC103KAT4A
- D2, D3: Manufacturer/Part Number (none) -> LL4002G; Supplier Stock Code (none) -> 821-LL4002G
- U2: Manufacturer/Part Number (none) -> LT1962EMS8-3.3#PBF; Supplier Stock Code (none) -> 584-1962EMS8-3.3PBF
- U3: Manufacturer/Part Number (none) -> LT3010EMS8E#PBF; Supplier Stock Code (none) -> 584-LT3010EMS8E#PBF
- U5, U6: Manufacturer/Part Number (none) -> LT1962EMS8-5#PBF; Supplier Stock Code (none) -> 584-LT1962EMS8-5#PBF

Commit message: update BOM
Parts:
- D7: Manufacturer/Part Number HSMG-C170 -> AP2012HD; Supplier Stock Code Mouser 630-HSMG-C170 -> 604-AP2012HD
Changed lines of the file:
@@
 F 2 "LED_SMD:LED_0805_2012Metric_Pad1.15x1.40mm_HandSolder" H 10250 2300 50  0001 C CNN
 F 3 "https://www.mouser.it/datasheet/2/678/av02-0551en-ds-hsmx-cxxx-05mar2012-1827675.pdf" H 10250 2300 50  0001 C CNN
-F 4 "HSMG-C170" H 10250 2300 50  0001 C CNN "Manufacturer/Part Number"
-F 5 "Mouser 630-HSMG-C170" H 10250 2300 50  0001 C CNN "Supplier Stock Code"
+F 4 "AP2012HD" H 10250 2300 50  0001 C CNN "Manufacturer/Part Number"
+F 5 "604-AP2012HD" H 10250 2300 50  0001 C CNN "Supplier Stock Code"
 	1    10250 2300
 	0    -1   -1   0

Commit message: update bom
Parts:
- D2, D3: Manufacturer/Part Number LL4002G -> SM4004-W; Supplier Stock Code 821-LL4002G -> 583-SM4004
- renumbered C16 to C14, C3 to C15, C5 to C16, C22 to C17, C23 to C18, C17 to C19, C19 to C20, C24 to C21, C21 to C22, C31 to C23, C32 to C24, C33 to C25, C34 to C26, C25 to C27, C35 to C28, C36 to C29, D7 to D4, J1 to J2, J2 to J3, R8 to R11, R11 to R12, R12 to R13, R13 to R14, U3 to U2, U2 to U3, U5 to U4, U6 to U5

Commit message: Update for DRC
Parts:
- D2, D3: footprint Diode_SMD:D_MELF -> Microwave_LO_Generator:D_MELF
- J2, J3: footprint Connector_PinHeader_2.54mm:PinHeader_1x02_P2.54mm_Vertical -> Microwave_LO_Generator:PinHeader_1x02_P2.54mm_Vertical
- TP2, TP3, TP4, TP5, TP6: footprint TestPoint:TestPoint_Loop_D2.60mm_Drill1.6mm_Beaded -> Microwave_LO_Generator:TestPoint_Loop_D2.60mm_Drill1.6mm_Beaded
- U2: footprint Package_SO:MSOP-8-1EP_3x3mm_P0.65mm_EP1.68x1.88mm -> Microwave_LO_Generator:MSOP-8-1EP_3x3mm_P0.65mm_EP1.68x1.88mm
- U3, U4, U5: footprint Package_SO:MSOP-8_3x3mm_P0.65mm -> Microwave_LO_Generator:MSOP-8_3x3mm_P0.65mm
Changed lines of the file:
@@
 F 0 "D2" V 1596 3822 50  0000 R CNN
 F 1 "DIODE" V 1505 3822 50  0000 R CNN
-F 2 "Diode_SMD:D_MELF" H 1550 3950 50  0001 C CNN
+F 2 "Microwave_LO_Generator:D_MELF" H 1550 3950 50  0001 C CNN
 F 3 "~" H 1550 3950 50  0001 C CNN
 F 4 "SM4004-W" V 1550 3950 50  0001 C CNN "Manufacturer/Part Number"
@@
 F 0 "U4" H 8800 3867 50  0000 C CNN
 F 1 "LT1962-5" H 8800 3776 50  0000 C CNN
-F 2 "Package_SO:MSOP-8_3x3mm_P0.65mm" H 8800 3050 50  0001 C CNN
+F 2 "Microwave_LO_Generator:MSOP-8_3x3mm_P0.65mm" H 8800 3050 50  0001 C CNN
 F 3 "https://www.analog.com/media/en/technical-documentation/data-sheets/1962fb.pdf" H 8800 2850 50  0001 C CNN
 F 4 "LT1962EMS8-5#PBF" H 8800 3400 50  0001 C CNN "Manufacturer/Part Number"
@@
 F 0 "U3" H 8700 2267 50  0000 C CNN
 F 1 "LT1962-3.3" H 8700 2176 50  0000 C CNN
-F 2 "Package_SO:MSOP-8_3x3mm_P0.65mm" H 8700 1450 50  0001 C CNN
+F 2 "Microwave_LO_Generator:MSOP-8_3x3mm_P0.65mm" H 8700 1450 50  0001 C CNN
 F 3 "https://www.analog.com/media/en/technical-documentation/data-sheets/1962fb.pdf" H 8700 1250 50  0001 C CNN
 F 4 "LT1962EMS8-3.3#PBF" H 8700 1800 50  0001 C CNN "Manufacturer/Part Number"
@@
 F 0 "U5" H 8800 5167 50  0000 C CNN
 F 1 "LT1962-5" H 8800 5076 50  0000 C CNN
-F 2 "Package_SO:MSOP-8_3x3mm_P0.65mm" H 8800 4350 50  0001 C CNN
+F 2 "Microwave_LO_Generator:MSOP-8_3x3mm_P0.65mm" H 8800 4350 50  0001 C CNN
 F 3 "https://www.analog.com/media/en/technical-documentation/data-sheets/1962fb.pdf" H 8800 4150 50  0001 C CNN
 F 4 "LT1962EMS8-5#PBF" H 8800 4700 50  0001 C CNN "Manufacturer/Part Number"
@@
 F 0 "U2" H 3250 4167 50  0000 C CNN
 F 1 "LT3010" H 3250 4076 50  0000 C CNN
-F 2 "Package_SO:MSOP-8-1EP_3x3mm_P0.65mm_EP1.68x1.88mm" H 3250 4125 50  0001 C CNN
+F 2 "Microwave_LO_Generator:MSOP-8-1EP_3x3mm_P0.65mm_EP1.68x1.88mm" H 3250 4125 50  0001 C CNN
 F 3 "https://www.analog.com/media/en/technical-documentation/data-sheets/30105fe.pdf" H 3250 3800 50  0001 C CNN
 F 4 "LT3010EMS8E#PBF" H 3250 3800 50  0001 C CNN "Manufacturer/Part Number"
@@
 F 0 "J2" H 1058 3881 50  0000 C CNN
 F 1 "Conn_01x02_Male" H 1058 3790 50  0000 C CNN
-F 2 "Connector_PinHeader_2.54mm:PinHeader_1x02_P2.54mm_Vertical" H 950 3700 50  0001 C CNN
+F 2 "Microwave_LO_Generator:PinHeader_1x02_P2.54mm_Vertical" H 950 3700 50  0001 C CNN
 F 3 "~" H 950 3700 50  0001 C CNN
 	1    950  3700
@@
 F 0 "J3" H 5658 1781 50  0000 C CNN
 F 1 "Conn_01x02_Male" H 5658 1690 50  0000 C CNN
-F 2 "Connector_PinHeader_2.54mm:PinHeader_1x02_P2.54mm_Vertical" H 5550 1600 50  0001 C CNN
+F 2 "Microwave_LO_Generator:PinHeader_1x02_P2.54mm_Vertical" H 5550 1600 50  0001 C CNN
 F 3 "~" H 5550 1600 50  0001 C CNN
 	1    5550 1600
@@
 F 0 "TP3" H 4958 3718 50  0000 L CNN
 F 1 "TestPoint" H 4958 3627 50  0000 L CNN
-F 2 "TestPoint:TestPoint_Loop_D2.60mm_Drill1.6mm_Beaded" H 5100 3600 50  0001 C CNN
+F 2 "Microwave_LO_Generator:TestPoint_Loop_D2.60mm_Drill1.6mm_Beaded" H 5100 3600 50  0001 C CNN
 F 3 "https://www.mouser.it/datasheet/2/215/005-5009-741293.pdf" H 5100 3600 50  0001 C CNN
 F 4 "5007" H 4900 3600 50  0001 C CNN "Manufacturer/Part Number"
@@
 F 0 "TP6" H 10308 1618 50  0000 L CNN
 F 1 "TestPoint" H 10308 1527 50  0000 L CNN
-F 2 "TestPoint:TestPoint_Loop_D2.60mm_Drill1.6mm_Beaded" H 10450 1500 50  0001 C CNN
+F 2 "Microwave_LO_Generator:TestPoint_Loop_D2.60mm_Drill1.6mm_Beaded" H 10450 1500 50  0001 C CNN
 F 3 "https://www.mouser.it/datasheet/2/215/005-5009-741293.pdf" H 10450 1500 50  0001 C CNN
 F 4 "5007" H 10250 1500 50  0001 C CNN "Manufacturer/Part Number"
@@
 F 0 "TP4" H 9958 3218 50  0000 L CNN
 F 1 "TestPoint" H 9958 3127 50  0000 L CNN
-F 2 "TestPoint:TestPoint_Loop_D2.60mm_Drill1.6mm_Beaded" H 10100 3100 50  0001 C CNN
+F 2 "Microwave_LO_Generator:TestPoint_Loop_D2.60mm_Drill1.6mm_Beaded" H 10100 3100 50  0001 C CNN
 F 3 "https://www.mouser.it/datasheet/2/215/005-5009-741293.pdf" H 10100 3100 50  0001 C CNN
 F 4 "5007" H 9900 3100 50  0001 C CNN "Manufacturer/Part Number"
@@
 F 0 "TP5" H 9958 4518 50  0000 L CNN
 F 1 "TestPoint" H 9958 4427 50  0000 L CNN
-F 2 "TestPoint:TestPoint_Loop_D2.60mm_Drill1.6mm_Beaded" H 10100 4400 50  0001 C CNN
+F 2 "Microwave_LO_Generator:TestPoint_Loop_D2.60mm_Drill1.6mm_Beaded" H 10100 4400 50  0001 C CNN
 F 3 "https://www.mouser.it/datasheet/2/215/005-5009-741293.pdf" H 10100 4400 50  0001 C CNN
 F 4 "5007" H 9900 4400 50  0001 C CNN "Manufacturer/Part Number"
@@
 F 0 "D3" V 6346 1722 50  0000 R CNN
 F 1 "DIODE" V 6255 1722 50  0000 R CNN
-F 2 "Diode_SMD:D_MELF" H 6300 1850 50  0001 C CNN
+F 2 "Microwave_LO_Generator:D_MELF" H 6300 1850 50  0001 C CNN
 F 3 "~" H 6300 1850 50  0001 C CNN
 F 4 "SM4004-W" V 6300 1850 50  0001 C CNN "Manufacturer/Part Number"
@@
 F 0 "TP2" H 1658 5318 50  0000 L CNN
 F 1 "TestPoint" H 1658 5227 50  0000 L CNN
-F 2 "TestPoint:TestPoint_Loop_D2.60mm_Drill1.6mm_Beaded" H 1800 5200 50  0001 C CNN
+F 2 "Microwave_LO_Generator:TestPoint_Loop_D2.60mm_Drill1.6mm_Beaded" H 1800 5200 50  0001 C CNN
 F 3 "https://www.mouser.it/datasheet/2/215/005-5009-741293.pdf" H 1800 5200 50  0001 C CNN
 F 4 "5007" H 1600 5200 50  0001 C CNN "Manufacturer/Part Number"
